Commit message: update.

File: gripper/gripper_description/urdf/gripper.urdf.xacro (robot description, xacro)
@@ -50,9 +50,36 @@
         <origin xyz="0 0 0" rpy="0 0 0"/>
         <geometry>
-          <mesh filename="package://gripper_description/meshes/base_link.stl"
-            scale="${stl_scale} ${stl_scale} ${stl_scale}"/>
-        </geometry>
-      </collision>
-    </link>
+          <mesh filename="package://gripper_description/meshes/base_link_old.stl"
+            scale="${stl_scale} ${stl_scale} ${stl_scale}"/>
+        </geometry>
+      </collision>
+    </link>
+    <link name="${prefix}gripper_motor">
+      <inertial>
+        <origin xyz="0 0 0" rpy="0 0 0"/>
+        <mass value="0.001"/>
+        <box_inertia m="0.001" x="0.05" y="0.05" z="0.05"/>
+      </inertial>
+      <visual>
+        <origin xyz="0 0 0" rpy="0 0 0"/>
+        <geometry>
+          <box size="0.05 0.04 0.05"/>
+        </geometry>
+       <material name="Cyan">
+         <color rgba="0.7 0.7 0.7 1.0"/>
+       </material>
+      </visual>
+      <collision>
+        <origin xyz="0 0 0" rpy="0 0 0"/>
+        <geometry>
+          <box size="0.05 0.04 0.05"/>
+        </geometry>
+      </collision>
+    </link>
+    <joint name="${prefix}gripper_motor_joint" type="fixed">
+      <parent link="${prefix}base_link"/>
+      <child link="${prefix}gripper_motor"/>
+      <origin xyz="0 -0.028 -0.08" rpy="0 0 0"/>
+    </joint>
     <joint name="${prefix}base_link_link_1_joint" type="fixed">
       <parent link="${prefix}base_link"/>

File: trex_description/urdf/trex.xacro (robot description, xacro)
@@ -226,5 +226,5 @@
       <parent link="base_link"/>
       <child link="hokuyo"/>
-      <origin xyz="0.6 0 0.2" rpy="3.14 0 0"/>
+      <origin xyz="0.6 0 0.2" rpy="0 0 0"/>
     </joint>
 <!--############################################UR5##################################################-->

Commit message: Updated gazebo simulation.

File: gripper/gripper_description/urdf/gripper.urdf.xacro (robot description, xacro)
@@ -193,5 +193,5 @@
     </link>
     <joint name="${prefix}base_link_camera_joint" type="fixed">
-      <origin xyz="0 0.025 0" rpy="3.14 0 1.57"/>
+      <origin xyz="0 0.025 0" rpy="0.0 0 1.57"/>
       <parent link="${prefix}base_link"/>
       <child link="${prefix}camera_link"/>

File: gripper/gripper_gazebo/urdf/gripper.gazebo.xacro (robot description, xacro)
@@ -54,5 +54,5 @@
     <gazebo reference="${prefix}_link">
       <sensor type="camera" name="${prefix}">
-        <update_rate>30.0</update_rate>
+        <update_rate>5.0</update_rate>
         <camera name="${prefix}">
           <horizontal_fov>1.5708</horizontal_fov>
